File: 7seg.kicad_pcb (KiCad board)
At the start: 2 copper layers, 12.4 x 15.2 mm, 12 parts, among them J1 Conn_01x05, J2 Conn_01x05, U1 74HC595, U2 HDSP-7401

Commit message: Add files via upload
Parts:
- added C1: C, Capacitors_SMD:C_0402, F.Cu at (101.0, 49.9)
- R1, R2, R3, R5, R6, R7, R8: value R -> 470
Routing:
- net (no net): track 0.00 -> 20.4 mm, vias 0 -> 2
- net Net-(R1-Pad2): track 1.06 -> 5.63 mm
- net Net-(R6-Pad1): track 4.79 -> 8.86 mm
- net Net-(R4-Pad1): track 8.74 -> 12.5 mm
- net Net-(R5-Pad1): track 8.53 -> 6.30 mm
- net Net-(J1-Pad3): track 24.6 -> 22.3 mm
- net VCC: track 19.6 -> 21.8 mm, vias 2 -> 1
- net GND: track 38.2 -> 36.3 mm
- net Net-(R2-Pad1): track 13.5 -> 15.3 mm
- net Net-(R7-Pad1): track 3.90 -> 5.31 mm
- net Net-(J2-Pad2): track 4.50 -> 5.62 mm
- net Net-(R8-Pad1): track 15.9 -> 14.9 mm
- net Net-(R1-Pad1): track 5.16 -> 4.27 mm
- net Net-(J1-Pad2): track 6.84 -> 6.17 mm
- net Net-(R3-Pad1): track 20.1 -> 20.7 mm
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- added copper zone on B.Cu, net GND
- added copper zone on B.Cu, net VCC
Other:
- board size 12.4 x 15.2 mm -> 12.3 x 18.8 mm
