File: 7seg.sch (KiCad schematic (older format))
At the start: 12 parts, among them J1 Conn_01x05, J2 Conn_01x05, U1 74HC595, U2 HDSP-7401

Commit message: Add files via upload
Parts:
- added C1: C, Capacitors_SMD:C_0402, symbol Device:C
- R1, R2, R3, R5, R6, R7, R8: value R -> 470
Connections:
- net GND: now also C1.2
- net VCC: now also C1.1
Other:
- moved on the sheet: J1, J2, R1, R2, R3, R4, R5, R6, R7, R8, U2

Commit message: Add files via upload
Parts:
- C1: value C -> 1u
Changed lines of the file:
@@
 P 2900 2400
 F 0 "C1" H 3015 2446 50  0000 L CNN
-F 1 "C" H 3015 2355 50  0000 L CNN
+F 1 "1u" H 3015 2355 50  0000 L CNN
 F 2 "Capacitors_SMD:C_0402" H 2938 2250 50  0001 C CNN
 F 3 "" H 2900 2400 50  0001 C CNN
